Commit message: ur5 urdf stl

File: ur5_description/urdf/ur5_gripper.urdf (robot description, URDF)
Before this commit: robot ur5, 24 links, 23 joints
Links:
- link forearm_link: geometry collision mesh filename=package://ur5_description/meshes/collision/forearm.stl; visual mesh filename=package://ur5_description/meshes/visual/forearm.dae
- link robot_base_link: geometry collision mesh filename=package://ur5_description/meshes/collision/base.stl; visual mesh filename=package://ur5_description/meshes/visual/base.dae
- link shoulder_link: geometry collision mesh filename=package://ur5_description/meshes/collision/shoulder.stl; visual mesh filename=package://ur5_description/meshes/visual/shoulder.dae
- link upper_arm_link: geometry collision mesh filename=package://ur5_description/meshes/collision/upperarm.stl; visual mesh filename=package://ur5_description/meshes/visual/upperarm.dae
- link wrist_1_link: geometry collision mesh filename=package://ur5_description/meshes/collision/wrist1.stl; visual mesh filename=package://ur5_description/meshes/visual/wrist1.dae
- link wrist_2_link: geometry collision mesh filename=package://ur5_description/meshes/collision/wrist2.stl; visual mesh filename=package://ur5_description/meshes/visual/wrist2.dae
- link wrist_3_link: geometry collision mesh filename=package://ur5_description/meshes/collision/wrist3.stl; visual mesh filename=package://ur5_description/meshes/visual/wrist3.dae

Commit message: revert ur5 urdf

File: ur5_description/urdf/ur5_gripper.urdf (robot description, URDF)
Before this commit: robot ur5, 24 links, 23 joints
Links:
- link forearm_link: geometry collision mesh filename=package://ur5_description/meshes/collision/forearm.dae; visual mesh filename=package://ur5_description/meshes/visual/forearm.dae
- link robot_base_link: geometry collision mesh filename=package://ur5_description/meshes/collision/base.dae; visual mesh filename=package://ur5_description/meshes/visual/base.dae
- link shoulder_link: geometry collision mesh filename=package://ur5_description/meshes/collision/shoulder.dae; visual mesh filename=package://ur5_description/meshes/visual/shoulder.dae
- link upper_arm_link: geometry collision mesh filename=package://ur5_description/meshes/collision/upperarm.dae; visual mesh filename=package://ur5_description/meshes/visual/upperarm.dae
- link wrist_1_link: geometry collision mesh filename=package://ur5_description/meshes/collision/wrist1.dae; visual mesh filename=package://ur5_description/meshes/visual/wrist1.dae
- link wrist_2_link: geometry collision mesh filename=package://ur5_description/meshes/collision/wrist2.dae; visual mesh filename=package://ur5_description/meshes/visual/wrist2.dae
- link wrist_3_link: geometry collision mesh filename=package://ur5_description/meshes/collision/wrist3.dae; visual mesh filename=package://ur5_description/meshes/visual/wrist3.dae
