Commit message: update spot urdf

File: robot_descriptions/spot_description/urdf/spot_arm.urdf (robot description, URDF)
Before this commit: robot spot_arm, 27 links, 26 joints
Links:
- link base_arm_link: geometry collision mesh filename=package://spot_arm/meshes/arm/base_link.dae scale=0.001 0.001 0.001; visual mesh filename=package://spot_arm/meshes/arm/base_link.dae scale=0.001 0.001 0.001
- link body: geometry collision mesh filename=package://spot_arm/meshes/body_collision.dae; visual mesh filename=package://spot_arm/meshes/body.dae
- link finger: geometry collision mesh filename=package://spot_arm/meshes/arm/finger.dae scale=0.001 0.001 0.001; visual mesh filename=package://spot_arm/meshes/arm/finger.dae scale=0.001 0.001 0.001
- link front_left_hip: geometry collision mesh filename=package://spot_arm/meshes/front_left_hip_collision.dae; visual mesh filename=package://spot_arm/meshes/front_left_hip.dae
- link front_left_lower_leg: geometry collision mesh filename=package://spot_arm/meshes/front_left_lower_leg_collision.dae; visual mesh filename=package://spot_arm/meshes/front_left_lower_leg.dae
- link front_left_upper_leg: geometry collision mesh filename=package://spot_arm/meshes/front_left_upper_leg_collision.dae; visual mesh filename=package://spot_arm/meshes/front_left_upper_leg.dae
- link front_right_hip: geometry collision mesh filename=package://spot_arm/meshes/front_right_hip_collision.dae; visual mesh filename=package://spot_arm/meshes/front_right_hip.dae
- link front_right_lower_leg: geometry collision mesh filename=package://spot_arm/meshes/front_right_lower_leg_collision.d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; visual mesh filename=package://spot_arm/meshes/front_right_lower_leg.dae
- link front_right_upper_leg: geometry collision mesh filename=package://spot_arm/meshes/front_right_upper_leg_collision.d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; visual mesh filename=package://spot_arm/meshes/front_right_upper_leg.dae
- link gripper: geometry collision mesh filename=package://spot_arm/meshes/arm/gripper.dae scale=0.001 0.001 0.001; visual mesh filename=package://spot_arm/meshes/arm/gripper.dae scale=0.001 0.001 0.001
- link link1: geometry collision mesh filename=package://spot_arm/meshes/arm/link1.dae scale=0.001 0.001 0.001; visual mesh filename=package://spot_arm/meshes/arm/link1.dae scale=0.001 0.001 0.001
- link link2: geometry collision mesh filename=package://spot_arm/meshes/arm/link2.dae scale=0.001 0.001 0.001; visual mesh filename=package://spot_arm/meshes/arm/link2.dae scale=0.001 0.001 0.001
- link link3: geometry collision mesh filename=package://spot_arm/meshes/arm/link3.dae scale=0.001 0.001 0.001; visual mesh filename=package://spot_arm/meshes/arm/link3.dae scale=0.001 0.001 0.001
- link link4: geometry collision mesh filename=package://spot_arm/meshes/arm/link4.dae scale=0.001 0.001 0.001; visual mesh filename=package://spot_arm/meshes/arm/link4.dae scale=0.001 0.001 0.001
- link rear_left_hip: geometry collision mesh filename=package://spot_arm/meshes/rear_left_hip_collision.dae; visual mesh filename=package://spot_arm/meshes/rear_left_hip.dae
- link rear_left_lower_leg: geometry collision mesh filename=package://spot_arm/meshes/rear_left_lower_leg_collision.dae; visual mesh filename=package://spot_arm/meshes/rear_left_lower_leg.dae
- link rear_left_upper_leg: geometry collision mesh filename=package://spot_arm/meshes/rear_left_upper_leg_collision.dae; visual mesh filename=package://spot_arm/meshes/rear_left_upper_leg.dae
- link rear_right_hip: geometry collision mesh filename=package://spot_arm/meshes/rear_right_hip_collision.dae; visual mesh filename=package://spot_arm/meshes/rear_right_hip.dae
- link rear_right_lower_leg: geometry collision mesh filename=package://spot_arm/meshes/rear_right_lower_leg_collision.dae; visual mesh filename=package://spot_arm/meshes/rear_right_lower_leg.dae
- link rear_right_upper_leg: geometry collision mesh filename=package://spot_arm/meshes/rear_right_upper_leg_collision.dae; visual mesh filename=package://spot_arm/meshes/rear_right_upper_leg.dae
- link wrist: geometry collision mesh filename=package://spot_arm/meshes/arm/wrist.dae scale=0.001 0.001 0.001; visual mesh filename=package://spot_arm/meshes/arm/wrist.dae scale=0.001 0.001 0.001
