Commit message: new ur5 urdf

File: robot_descriptions/ur5_description/urdf/ur5_gripper.urdf (robot description, URDF)
Before this commit: robot ur5, 24 links, 23 joints
Links:
- removed link ee_link
- removed link pedestal
- removed link robot_base_link
- added link base_link_inertia, mass 4.0; collision mesh filename=package://ur5_description/meshes/collision/base.dae; visual mesh filename=package://ur5_description/meshes/visual/base.dae
- added link flange
Joints:
- removed joint ee_fixed_joint
- removed joint pedestal_joint
- removed joint robot_base_joint
- removed joint wrist_3_link-tool0_fixed_joint
- added joint base_link-base_link_inertia: type fixed, parent base_link, child base_link_inertia, origin xyz=0 0 0 rpy=0 0 3.14159265359
- added joint flange-tool0: type fixed, parent flange, child tool0, origin xyz=0 0 0 rpy=1.57079632679 0 1.57079632679
- added joint wrist_3-flange: type fixed, parent wrist_3_link, child flange, origin xyz=0 0 0 rpy=0 -1.57079632679 -1.57079632679
- joint base_link-base_fixed_joint: origin xyz=0 0 0 rpy=0 0 -3.14159265359 -> xyz=0 0 0 rpy=0 0 3.14159265359
- joint elbow_joint: axis 0 1 0 -> 0 0 1; limit lower=-6.2831853 upper=6.2831853 effort=150.0 velocity=3.15 -> lower=-3.14159265359 upper=3.14159265359 effort=150.0 velocity=3.14159265359; origin xyz=0.0 -0.1197 0.425 rpy=0.0 0.0 0.0 -> xyz=-0.4251354753856735 0 0 rpy=0 0 0
- joint finger_tip_joint: origin xyz= 0.0 0.2323 0.0 rpy=-1.57079632679 0.0 0.0 -> xyz= 0.0 0.0 0.15 rpy=0.0 0.0 0.0
- joint shoulder_lift_joint: axis 0 1 0 -> 0 0 1; limit lower=-6.2831853 upper=6.2831853 effort=150.0 velocity=3.15 -> lower=-6.28318530718 upper=6.28318530718 effort=150.0 velocity=3.14159265359; origin xyz=0.0 0.13585 0.0 rpy=0.0 0.0 0.0 -> xyz=0.0001345759894064394 0 0 rpy=1.57114841778325 0 0
- joint shoulder_pan_joint: limit lower=-6.2831853 upper=6.2831853 effort=150.0 velocity=3.15 -> lower=-6.28318530718 upper=6.28318530718 effort=150.0 velocity=3.14159265359; origin xyz=0.0 0.0 0.089159 rpy=0.0 0.0 0.0 -> xyz=0 0 0.0894297563087571 rpy=0 0 0; parent robot_base_link -> base_link_inertia
- joint ur5_ee_link-gripper_base: origin xyz= 0.0 0.0 0.0 rpy=0.0 1.57079632679 0.0 -> xyz= 0.0 0.0 0.0 rpy=0.0 0.0 0.0; parent ee_link -> tool0
- joint wrist_1_joint: axis 0 1 0 -> 0 0 1; limit lower=-6.2831853 upper=6.2831853 effort=28.0 velocity=3.2 -> lower=-6.28318530718 upper=6.28318530718 effort=28.0 velocity=3.14159265359; origin xyz=0.0 0.0 0.39225 rpy=0.0 0.0 0.0 -> xyz=-0.3920852041618563 0.00156975446298503 0.1104928652798279 rpy=0 0 0
- joint wrist_2_joint: limit lower=-6.2831853 upper=6.2831853 effort=28.0 velocity=3.2 -> lower=-6.28318530718 upper=6.28318530718 effort=28.0 velocity=3.14159265359; origin xyz=0.0 0.093 0.0 rpy=0.0 0.0 0.0 -> xyz=0 -0.09483720192826969 0.0 rpy=1.570239865752715 0 0
- joint wrist_3_joint: axis 0 1 0 -> 0 0 1; limit lower=-6.2831853 upper=6.2831853 effort=28.0 velocity=3.2 -> lower=-6.28318530718 upper=6.28318530718 effort=28.0 velocity=3.14159265359; origin xyz=0.0 0.0 0.09465 rpy=0.0 0.0 0.0 -> xyz=0 0.0824592599587561 0.0 rpy=1.571751493258682 3.141592653589793 -3.141559191090251
