Commit message: Spot URDF body test

File: robot_descriptions/spot_arm/urdf/spot_arm.urdf (robot description, URDF)
Before this commit: robot spot_arm, 27 links, 26 joints
Links:
- link body: geometry collision mesh filename=package://spot_arm/meshes/body_collision.dae; visual mesh filename=package://spot_arm/meshes/body_collision.dae

Commit message: Spot Body Material Test

File: robot_descriptions/spot_arm/urdf/spot_arm.urdf (robot description, URDF)
Before this commit: robot spot_arm, 27 links, 26 joints
Links:
- link body: geometry collision mesh filename=package://spot_arm/meshes/body_collision.dae; visual mesh filename=package://spot_arm/meshes/body.dae

Commit message: Switch Spot Parts Test

File: robot_descriptions/spot_arm/urdf/spot_arm.urdf (robot description, URDF)
Before this commit: robot spot_arm, 27 links, 26 joints
Links:
- link body: geometry collision mesh filename=package://spot_arm/meshes/body_collision.dae; visual mesh filename=package://spot_arm/meshes/front_left_upper_leg.dae
- link front_left_upper_leg: geometry collision mesh filename=package://spot_arm/meshes/front_left_upper_leg_collision.dae; visual mesh filename=package://spot_arm/meshes/body.dae

Commit message: Switch Spot Parts Back

File: robot_descriptions/spot_arm/urdf/spot_arm.urdf (robot description, URDF)
Before this commit: robot spot_arm, 27 links, 26 joints
Links:
- link body: geometry collision mesh filename=package://spot_arm/meshes/body_collision.dae; visual mesh filename=package://spot_arm/meshes/body.dae
- link front_left_upper_leg: geometry collision mesh filename=package://spot_arm/meshes/front_left_upper_leg_collision.dae; visual mesh filename=package://spot_arm/meshes/front_left_upper_leg.dae

Commit message: Spot Base Link Collision

File: robot_descriptions/spot_arm/urdf/spot_arm.urdf (robot description, URDF)
Before this commit: robot spot_arm, 27 links, 26 joints
Links:
- link base_arm_link: geometry collision mesh filename=package://spot_arm/meshes/arm/base_link_collision.dae scale=0.001 0.001 0.001; visual mesh filename=package://spot_arm/meshes/arm/base_link.dae scale=0.001 0.001 0.001

Commit message: Spot Base URDF Resize

File: robot_descriptions/spot_arm/urdf/spot_arm.urdf (robot description, URDF)
Before this commit: robot spot_arm, 27 links, 26 joints
Links:
- link base_arm_link: geometry collision mesh filename=package://spot_arm/meshes/arm/base_link_collision.dae scale=0.1 0.1 0.1; visual mesh filename=package://spot_arm/meshes/arm/base_link.dae scale=0.1 0.1 0.1

Commit message: Spot URDF New Visual Geometry

File: robot_descriptions/spot_arm/urdf/spot_arm.urdf (robot description, URDF)
Before this commit: robot spot_arm, 27 links, 26 joints
Links:
- link finger: geometry collision mesh filename=package://spot_arm/meshes/arm/finger_collision.dae scale=0.1 0.1 0.1; visual mesh filename=package://spot_arm/meshes/arm/finger.dae scale=0.1 0.1 0.1
- link gripper: geometry collision mesh filename=package://spot_arm/meshes/arm/gripper_collision.dae scale=0.1 0.1 0.1; visual mesh filename=package://spot_arm/meshes/arm/gripper.dae scale=0.1 0.1 0.1
- link link1: geometry collision mesh filename=package://spot_arm/meshes/arm/link1_collision.dae scale=0.1 0.1 0.1; visual mesh filename=package://spot_arm/meshes/arm/link1.dae scale=0.1 0.1 0.1
- link link2: geometry collision mesh filename=package://spot_arm/meshes/arm/link2_collision.dae scale=0.1 0.1 0.1; visual mesh filename=package://spot_arm/meshes/arm/link2.dae scale=0.1 0.1 0.1
- link link3: geometry collision mesh filename=package://spot_arm/meshes/arm/link3_collision.dae scale=0.1 0.1 0.1; visual mesh filename=package://spot_arm/meshes/arm/link3.dae scale=0.1 0.1 0.1
- link link4: geometry collision mesh filename=package://spot_arm/meshes/arm/link4_collision.dae scale=0.1 0.1 0.1; visual mesh filename=package://spot_arm/meshes/arm/link4.dae scale=0.1 0.1 0.1
- link wrist: geometry collision mesh filename=package://spot_arm/meshes/arm/wrist_collision.dae scale=0.1 0.1 0.1; visual mesh filename=package://spot_arm/meshes/arm/wrist.dae scale=0.1 0.1 0.1

Commit message: Spot URDF Default Leg Joints

File: robot_descriptions/spot_arm/urdf/spot_arm.urdf (robot description, URDF)
Before this commit: robot spot_arm, 27 links, 26 joints
Joints:
- joint front_left_hip_y: origin xyz=0.0 0.110945 0.0 rpy=0 1.3 0 -> xyz=0.0 0.110945 0.0 rpy=0 1.0 0
- joint front_left_knee: origin xyz=0.025 0.000 -0.3205 rpy=0 -2.6 0 -> xyz=0.025 0.000 -0.3205 rpy=0 -2.0 0
- joint front_right_hip_y: origin xyz=0.0 -0.110945 0.0 rpy=0 1.3 0 -> xyz=0.0 -0.110945 0.0 rpy=0 1.0 0
- joint front_right_knee: origin xyz=0.025 0.000 -0.3205 rpy=0 -2.6 0 -> xyz=0.025 0.000 -0.3205 rpy=0 -2.0 0
- joint rear_left_hip_y: origin xyz=0.0 0.110945 0.0 rpy=0 1.3 0 -> xyz=0.0 0.110945 0.0 rpy=0 1.0 0
- joint rear_left_knee: origin xyz=0.025 0.000 -0.3205 rpy=0 -2.6 0 -> xyz=0.025 0.000 -0.3205 rpy=0 -2.0 0
- joint rear_right_hip_y: origin xyz=0.0 -0.110945 0.0 rpy=0 1.3 0 -> xyz=0.0 -0.110945 0.0 rpy=0 1.0 0
- joint rear_right_knee: origin xyz=0.025 0.000 -0.3205 rpy=0 -2.6 0 -> xyz=0.025 0.000 -0.3205 rpy=0 -2.0 0
